Commit message: Fix base_footprint position and test_room pose in the world file
- testbed.xacro: base_footprint sat 6 cm from the wheel-axle midpoint, so
  spinning in place looked like sideways motion to AMCL (error up to 0.51 m
  after one spin). Move it to the axle midpoint; AMCL error is now 2-7 cm.
- testbed_playground.world: the test_room model's definition pose disagreed
  with its saved <state> pose by 1.25 m, so Reset World moved every brick
  wall off the map. Set the definition pose to the state pose.

File: testbed_description/urdf/testbed.xacro (robot description, xacro)
@@ -215,5 +215,5 @@
   <parent link="base_footprint" />
   <child link="base_link" />
-  <origin xyz="0 0 0" rpy="0 0 0" />
+  <origin xyz="0.0505 0.0378 0" rpy="0 0 0" />
 </joint>
 <joint name="left_wheel_joint" type="continuous">
